File: hw/pulser_frontend/MAGIE_pulser_frontend.kicad_pcb (KiCad board)
At the start: 8 copper layers, 220 x 120.1 mm, 1649 parts, among them J1 45558-0003, J10 Header male 2x05, J12 Header male 2x05, J13 Header male 1x02, J14 Header male 2x03, J15 Header male 2x03, J16 Header male 2x03, J17 Header male 2x03, J18 Header male 1x02, J19 PCIe x8, J2 Header male 2x05, J20 Header male 1x02, J21 Header male 1x02, J22 Header male 1x02, J3 Header male 1x02, J4 PCIe x16 card, J5 Header male 2x02, J6 Header male 2x02, J7 Header male 2x03, J8 Header male 2x03, J9 Header male 2x03, Q1 DMG2302UK, Q2 DMG2302UK, Q3 DMG2302UK, Q4 DMG2302UK, Q5 DMG2302UK, Q6 MMBT3906-7-F, U1 LMK00304SQ, U10 TPSM64406RCHR, U11 TPSM64406RCHR, U12 TPSM64406RCHR, U13 TPS63710, U14 TPS7A9601, U15 TPS7A9601, U18 TPS7A9601, U19 TPS7A9601, U2 LMK1C1104DQF, U20 MAX38902A, U21 MAX38902A, U23 TCA9800DGKR, U24 SN74AUC1G32DBVR, U3 74LVC1G06GW, U4 LMK00304SQ, U5 SN65LVDS104PW, U6 BTS5030-1EJA, U7 74LVC1G11GW-Q100, U9 LM3880MF-1AE

Commit message: Update MAGIE ultrasound Frontend board for manufacturing
Routing:
- net /Channel group 3/P_HVP0: track 21.8 -> 22.0 mm, vias 12 -> 13
- net Net-(U13-SW): vias 2 -> 4
- net /P_M3V3A: vias 19 -> 21
