File: hw/pulser_frontend/MAGIE_pulser_frontend.kicad_sch (KiCad schematic)
At the start: 15 parts, among them J1 45558-0003, J20 Header male 1x02, J21 Header male 1x02, J22 Header male 1x02, J3 Header male 1x02

Commit message: Update MAGIE ultrasound Frontend board for manufacturing
Changed lines of the file:
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@@
 	(wire
 		(pts
-			(xy 266.7 209.55) (xy 283.21 209.55)
+			(xy 266.7 210.82) (xy 283.21 210.82)
 		)
 		(stroke
@@
 	)
 	(label "PLS_DATAOUT3"
-		(at 283.21 209.55 180)
+		(at 283.21 210.82 180)
 		(effects
 			(font
@@
 		)
 		(pin "DATAOUT" output
-			(at 266.7 209.55 0)
+			(at 266.7 210.82 0)
 			(effects
 				(font
